File: eagle/atmega_midi_pg800.brd (EAGLE design)
At the start: 100 x 80.8 mm, 39 parts, among them IC1 78L05Z, IC2 4067N, IC3 4067N, IC4 4067N, Q1 16.000Mhz, U1 6N138, U2 ATMEGA328P_PDIP, X1 MAB6H

Commit message: placed again
Parts:
- moved IN16 84.6 mm to (74.9, 33.0), turned to 270 degrees
Other:
- board size 100 x 80.8 mm -> 100 x 80 mm
Changed lines of the file:
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@@
 <wire x1="100" y1="80" x2="0" y2="80" width="0" layer="20"/>
 <wire x1="0" y1="80" x2="0" y2="0" width="0" layer="20"/>
-<wire x1="74.422" y1="-0.762" x2="2.794" y2="-0.762" width="1.6764" layer="46"/>
 <wire x1="48.514" y1="6.096" x2="49.276" y2="6.096" width="1.6764" layer="46"/>
 <wire x1="49.276" y1="6.096" x2="49.276" y2="4.826" width="1.6764" layer="46"/>
@@
 <attribute name="OC_FARNELL" value="1462920" x="12.7" y="43.18" size="1.778" layer="27" display="off"/>
 </element>
-<element name="IN16" library="con-molex" package="22-23-2041" value="22-23-2041" x="6.35" y="-16.51">
-<attribute name="MF" value="MOLEX" x="6.35" y="-16.51" size="1.778" layer="27" display="off"/>
-<attribute name="MPN" value="22-23-2041" x="6.35" y="-16.51" size="1.778" layer="27" display="off"/>
-<attribute name="OC_NEWARK" value="38C0355" x="6.35" y="-16.51" size="1.778" layer="27" display="off"/>
-<attribute name="OC_FARNELL" value="1462920" x="6.35" y="-16.51" size="1.778" layer="27" display="off"/>
+<element name="IN16" library="con-molex" package="22-23-2041" value="22-23-2041" x="74.93" y="33.02" rot="R270">
+<attribute name="MF" value="MOLEX" x="74.93" y="33.02" size="1.778" layer="27" rot="R270" display="off"/>
+<attribute name="MPN" value="22-23-2041" x="74.93" y="33.02" size="1.778" layer="27" rot="R270" display="off"/>
+<attribute name="OC_NEWARK" value="38C0355" x="74.93" y="33.02" size="1.778" layer="27" rot="R270" display="off"/>
+<attribute name="OC_FARNELL" value="1462920" x="74.93" y="33.02" size="1.778" layer="27" rot="R270" display="off"/>
 </element>
 </elements>
@@
 <contactref element="U2" pad="14"/>
 <contactref element="IN16" pad="1"/>
-<wire x1="2.54" y1="-16.51" x2="68.58" y2="29.21" width="0" layer="19" extent="1-1"/>
+<wire x1="74.93" y1="36.83" x2="68.58" y2="29.21" width="0" layer="19" extent="1-1"/>
 </signal>
 <signal name="N$17">
 <contactref element="U2" pad="15"/>
 <contactref element="IN16" pad="2"/>
-<wire x1="5.08" y1="-16.51" x2="68.58" y2="36.83" width="0" layer="19" extent="1-1"/>
+<wire x1="74.93" y1="34.29" x2="68.58" y2="36.83" width="0" layer="19" extent="1-1"/>
 </signal>
 <signal name="N$77">
 <contactref element="U2" pad="16"/>
 <contactref element="IN16" pad="3"/>
-<wire x1="7.62" y1="-16.51" x2="66.04" y2="36.83" width="0" layer="19" extent="1-1"/>
+<wire x1="74.93" y1="31.75" x2="66.04" y2="36.83" width="0" layer="19" extent="1-1"/>
 </signal>
 <signal name="N$78">
 <contactref element="U2" pad="17"/>
 <contactref element="IN16" pad="4"/>
-<wire x1="10.16" y1="-16.51" x2="63.5" y2="36.83" width="0" layer="19" extent="1-1"/>
+<wire x1="74.93" y1="29.21" x2="63.5" y2="36.83" width="0" layer="19" extent="1-1"/>
 </signal>
 </signals>
