File: eagle/vco_pots.brd (EAGLE design)
At the start: 100 x 80 mm, 17 parts, among them P1 P0915N, P10 P0915N, P2 P0915N, P3 P0915N, P4 P0915N, P5 P0915N, P6 P0915N, P7 P0915N, P8 P0915N, P9 P0915N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

Commit message: schemo wired
Parts:
- removed X1: 87758-1416, con-molex:87758-1416
- added JP1, JP2: (no value), pinhead:1X07
- moved X3 52.1 mm to (8.89, 72.4), turned to 270 degrees
- moved X2 48.3 mm to (8.89, 68.6), turned to 270 degrees
- moved P10 17.8 mm to (12.7, 35.6)
- moved P6 17.8 mm to (50.8, 49.5)
- moved P7 17.8 mm to (50.8, 35.6)
- moved P9 17.8 mm to (12.7, 49.5)
- moved P5 17.8 mm to (50.8, 21.6)
- moved P8 17.8 mm to (12.7, 21.6)
- moved P1 4.02 mm to (88.9, 63.5)
- moved P3 4.02 mm to (88.9, 49.5)
- moved P2 4.02 mm to (88.9, 21.6)
- moved P4 4.02 mm to (88.9, 35.6)
- moved TM2 2.84 mm to (63.5, 44.5)
- moved TM3 2.84 mm to (38.1, 44.5)
- moved TM4 2.84 mm to (25.4, 44.5)
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Connections:
- new net N$11: JP1.4, TM4.WIPER
- new net N$12: JP1.5, TM3.WIPER
- new net N$13: JP2.2, TM2.WIPER
- new net N$14: JP2.3, TM1.WIPER
- new net N$6: JP1.1, P8.S
- net N$1: now also JP1.2
- net N$10: now also JP2.4
- net N$2: now also JP2.1
- net N$3: now also JP2.5
- net N$4: now also JP1.6
- net N$5: now also JP2.6
- net N$7: now also JP1.3
- net N$8: now also JP1.7
- net N$9: now also JP2.7
